Commit message: Reconstruct the driver package

File: alicia_duo_descriptions/urdf/alicia_duo_with_gripper.urdf (robot description, URDF)
Before this commit: robot alicia_duo_descriptions, 11 links, 10 joints
Links:
- link Grasp_base: mass 0.0482959693358257 -> 0.13604884360545
- link Link1: mass 0.1961 -> 0.203075737500143
- link Link2: mass 0.21717 -> 0.228750683078605
- link Link3: mass 0.0865602005421272 -> 0.0902084989642731
- link Link4: mass 0.0943760430662397 -> 0.0791974889780253
- link Link5: mass 0.0298054906363541 -> 0.0472226666291309
- link Link6: mass 0.00075405362358679 -> 0.000754043064008528
- link Link7: mass 0.0298800419940728 -> 0.0243492837152759
- link Link8: mass 0.0298800419940728 -> 0.0243228050977196
Joints:
- joint Grasp2tool: origin xyz=-0.0065308 -0.00063845 0.11382 rpy=0 0 0 -> xyz=0.00275 0.0008332 0.13779 rpy=0 0 0
- joint Joint1: origin xyz=0 0 0.0745 rpy=0 0 0 -> xyz=0 0 0.1445 rpy=0 0 0
- joint Joint2: origin xyz=-4E-05 0 0.09361 rpy=-1.5708 -1.4701 0 -> xyz=0 0 0.025106 rpy=1.5708 -1.5708 0
- joint Joint3: origin xyz=0.22471 0 0.0004 rpy=0 0 -2.4569 -> xyz=0.22367 0.022494 -5E-05 rpy=0 0 2.3562
- joint Joint4: origin xyz=0.00211 -0.0969 -0.0005 rpy=1.5708 0 0 -> xyz=0.0988 0.00211 -0.0001 rpy=1.5708 0 1.5708
- joint Joint5: axis 0 0 1 -> 0 0 -1; origin xyz=0.00014 0.0002 0.12011 rpy=-1.5708 0 0 -> xyz=0 -0.0007 0.12011 rpy=-1.5708 0 0
- joint Joint6: origin xyz=-0.00389 -0.0592 0.00064 rpy=1.5708 0 0 -> xyz=-0.0038938 -0.0573 0.0008 rpy=1.5708 0 0
- joint left_finger: axis 0 0 -1 -> 0 0 0; limit (none) -> lower=-0.0125 upper=0 effort=5 velocity=10; origin xyz=-0.0065308 -0.015222 0.11382 rpy=1.5708 0 0 -> xyz=0.00275 -0.0011661 0.13779 rpy=1.5451 0 0
- joint right_finger: axis 0 0 1 -> 0 0 0; limit (none) -> lower=0 upper=0.0125 effort=5 velocity=10; origin xyz=-0.0065308 0.013945 0.11382 rpy=1.5708 0 3.1416 -> xyz=0.00275 0.0028325 0.13768 rpy=-1.5965 0 0

File: alicia_duo_moveit/config/alicia_duo_descriptions.ros2_control.xacro (robot description, xacro)
@@ -5,6 +5,6 @@
         <ros2_control name="${name}" type="system">
             <hardware>
-                <!-- By default, set up controllers for simulation. This won't work on real hardware -->
-                <plugin>mock_components/GenericSystem</plugin>
+                <!-- Use xacro:if/unless to select the plugin -->
+                <plugin>alicia_duo_hardware_interface/AliciaHardwareInterface</plugin>
             </hardware>
             <joint name="Joint1">
@@ -13,5 +13,5 @@
                   <param name="initial_value">${initial_positions['Joint1']}</param>
                 </state_interface>
-                <state_interface name="velocity"/>
+                <!-- <state_interface name="velocity"/> -->
             </joint>
             <joint name="Joint2">
@@ -20,5 +20,5 @@
                   <param name="initial_value">${initial_positions['Joint2']}</param>
                 </state_interface>
-                <state_interface name="velocity"/>
+                <!-- <state_interface name="velocity"/> -->
             </joint>
             <joint name="Joint3">
@@ -27,5 +27,5 @@
                   <param name="initial_value">${initial_positions['Joint3']}</param>
                 </state_interface>
-                <state_interface name="velocity"/>
+                <!-- <state_interface name="velocity"/> -->
             </joint>
             <joint name="Joint4">
@@ -34,5 +34,5 @@
                   <param name="initial_value">${initial_positions['Joint4']}</param>
                 </state_interface>
-                <state_interface name="velocity"/>
+                <!-- <state_interface name="velocity"/> -->
             </joint>
             <joint name="Joint5">
@@ -41,5 +41,5 @@
                   <param name="initial_value">${initial_positions['Joint5']}</param>
                 </state_interface>
-                <state_interface name="velocity"/>
+                <!-- <state_interface name="velocity"/> -->
             </joint>
             <joint name="Joint6">
@@ -48,5 +48,5 @@
                   <param name="initial_value">${initial_positions['Joint6']}</param>
                 </state_interface>
-                <state_interface name="velocity"/>
+                <!-- <state_interface name="velocity"/> -->
             </joint>
         </ros2_control>

File: alicia_duo_moveit/config/alicia_duo_descriptions.urdf.xacro (robot description, xacro)
@@ -2,8 +2,10 @@
 <robot xmlns:xacro="http://www.ros.org/wiki/xacro" name="alicia_duo_descriptions">
     <xacro:arg name="initial_positions_file" default="initial_positions.yaml" />
+    <xacro:arg name="use_fake_hardware" default="true" />
     <!-- Import alicia_duo_descriptions urdf file -->
     <xacro:include filename="$(find alicia_duo_descriptions)/urdf/alicia_duo_with_gripper.urdf" />
     <!-- Import control_xacro -->
     <xacro:include filename="alicia_duo_descriptions.ros2_control.xacro" />
-    <xacro:alicia_duo_descriptions_ros2_control name="FakeSystem" initial_positions_file="$(arg initial_positions_file)"/>
+    <!-- Pass the argument to the macro -->
+    <xacro:alicia_duo_descriptions_ros2_control name="AliciaDuoSystem" initial_positions_file="$(arg initial_positions_file)" use_fake_hardware="$(arg use_fake_hardware)"/>
 </robot>

Commit message: Update ros2 controller configuration

File: alicia_duo_descriptions/urdf/alicia_duo_with_gripper.urdf (robot description, URDF)
Before this commit: robot alicia_duo_descriptions, 11 links, 10 joints
Joints:
- joint left_finger: origin xyz=0.00275 -0.0011661 0.13779 rpy=1.5451 0 0 -> xyz=0.00275 -0.025 0.13779 rpy=1.5451 0 0; type fixed -> prismatic
- joint right_finger: mimic (none) -> joint=left_finger multiplier=-1 offset=0; origin xyz=0.00275 0.0028325 0.13768 rpy=-1.5965 0 0 -> xyz=0.00275 0.025 0.13768 rpy=-1.5965 0 0; type fixed -> prismatic

Commit message: Add gripper control moveit configuration

File: alicia_duo_descriptions/urdf/alicia_duo_with_gripper.urdf (robot description, URDF)
Before this commit: robot alicia_duo_descriptions, 11 links, 10 joints
Joints:
- joint left_finger: axis 0 0 0 -> 0 0 1; limit lower=-0.0125 upper=0 effort=5 velocity=10 -> lower=-0.022 upper=0 effort=5 velocity=10
- joint right_finger: axis 0 0 0 -> 0 0 -1; limit lower=0 upper=0.0125 effort=5 velocity=10 -> lower=0 upper=0.022 effort=5 velocity=10

File: aliciad_moveit/config/alicia_duo_descriptions.ros2_control.xacro (robot description, xacro)
@@ -5,5 +5,6 @@
         <ros2_control name="${name}" type="system">
             <hardware>
-                <!-- Use xacro:if/unless to select the plugin -->
+                <!-- By default, set up controllers for simulation. This won't work on real hardware -->
+                <!-- <plugin>mock_components/GenericSystem</plugin> -->
                 <plugin>alicia_duo_driver/AliciaHardwareInterface</plugin>
                 <param name="port">/dev/ttyUSB0</param>
@@ -16,5 +17,4 @@
                   <param name="initial_value">${initial_positions['Joint1']}</param>
                 </state_interface>
-                <!-- <state_interface name="velocity"/> -->
             </joint>
             <joint name="Joint2">
@@ -23,5 +23,4 @@
                   <param name="initial_value">${initial_positions['Joint2']}</param>
                 </state_interface>
-                <!-- <state_interface name="velocity"/> -->
             </joint>
             <joint name="Joint3">
@@ -30,5 +29,4 @@
                   <param name="initial_value">${initial_positions['Joint3']}</param>
                 </state_interface>
-                <!-- <state_interface name="velocity"/> -->
             </joint>
             <joint name="Joint4">
@@ -37,5 +35,4 @@
                   <param name="initial_value">${initial_positions['Joint4']}</param>
                 </state_interface>
-                <!-- <state_interface name="velocity"/> -->
             </joint>
             <joint name="Joint5">
@@ -44,5 +41,4 @@
                   <param name="initial_value">${initial_positions['Joint5']}</param>
                 </state_interface>
-                <!-- <state_interface name="velocity"/> -->
             </joint>
             <joint name="Joint6">
@@ -51,5 +47,10 @@
                   <param name="initial_value">${initial_positions['Joint6']}</param>
                 </state_interface>
-                <!-- <state_interface name="velocity"/> -->
+            </joint>
+            <joint name="left_finger">
+                <command_interface name="position"/>
+                <state_interface name="position">
+                  <param name="initial_value">${initial_positions['left_finger']}</param>
+                </state_interface>
             </joint>
         </ros2_control>

File: aliciad_moveit/config/alicia_duo_descriptions.urdf.xacro (robot description, xacro)
@@ -2,10 +2,9 @@
 <robot xmlns:xacro="http://www.ros.org/wiki/xacro" name="alicia_duo_descriptions">
     <xacro:arg name="initial_positions_file" default="initial_positions.yaml" />
-    <xacro:arg name="use_fake_hardware" default="false" />
     <!-- Import alicia_duo_descriptions urdf file -->
     <xacro:include filename="$(find alicia_duo_descriptions)/urdf/alicia_duo_with_gripper.urdf" />
     <!-- Import control_xacro -->
     <xacro:include filename="alicia_duo_descriptions.ros2_control.xacro" />
-    <!-- Pass the argument to the macro -->
+    <!-- <xacro:alicia_duo_descriptions_ros2_control name="FakeSystem" initial_positions_file="$(arg initial_positions_file)"/> -->
     <xacro:alicia_duo_descriptions_ros2_control name="AliciaDuoSystem" initial_positions_file="$(arg initial_positions_file)"/>
 </robot>

Commit message: Add ompl_planning setting

File: alicia_duo_descriptions/urdf/alicia_duo_with_gripper.urdf (robot description, URDF)
Before this commit: robot alicia_duo_descriptions, 11 links, 10 joints
Links:
- link Link7: geometry visual mesh filename=package://alicia_duo_descriptions/meshes/Link7.STL
- link Link8: geometry visual mesh filename=package://alicia_duo_descriptions/meshes/Link8.STL
Joints:
- removed joint Joint1
- removed joint Joint2
- removed joint Joint3
- removed joint Joint4
- removed joint Joint5
- removed joint Joint6
- removed joint Joint6_to_gripper_base
- added joint joint1: type revolute, parent base_link, child Link1, origin xyz=0 0 0.1445 rpy=0 0 0, axis 0 0 1, limit lower=-2.16 upper=2.16 effort=12 velocity=5
- added joint joint2: type revolute, parent Link1, child Link2, origin xyz=0 0 0.025106 rpy=1.5708 -1.5708 0, axis 0 0 -1, limit lower=-3.14 upper=3.14 effort=12 velocity=5
- added joint joint3: type revolute, parent Link2, child Link3, origin xyz=0.22367 0.022494 -5E-05 rpy=0 0 2.3562, axis 0 0 -1, limit lower=-3.14 upper=3.14 effort=12 velocity=5
- added joint joint4: type revolute, parent Link3, child Link4, origin xyz=0.0988 0.00211 -0.0001 rpy=1.5708 0 1.5708, axis 0 0 -1, limit lower=-3.14 upper=3.14 effort=12 velocity=5
- added joint joint5: type revolute, parent Link4, child Link5, origin xyz=0 -0.0007 0.12011 rpy=-1.5708 0 0, axis 0 0 -1, limit lower=-3.14 upper=3.14 effort=12 velocity=5
- added joint joint6: type revolute, parent Link5, child Link6, origin xyz=-0.0038938 -0.0573 0.0008 rpy=1.5708 0 0, axis 0 0 -1, limit lower=-3.14 upper=3.14 effort=12 velocity=5
- added joint joint6_to_gripper_base: type fixed, parent Link6, child Grasp_base, origin xyz=0 0 0 rpy=0 0 0, axis 0 0 0
- joint left_finger: mimic (none) -> joint=right_finger multiplier=-1 offset=0
- joint right_finger: mimic joint=left_finger multiplier=-1 offset=0 -> (none)

File: alicia_duo_moveit/config/alicia_duo_descriptions.ros2_control.xacro (robot description, xacro)
@@ -5,6 +5,4 @@
         <ros2_control name="${name}" type="system">
             <hardware>
-                <!-- By default, set up controllers for simulation. This won't work on real hardware -->
-                <!-- <plugin>mock_components/GenericSystem</plugin> -->
                 <plugin>alicia_duo_driver/AliciaHardwareInterface</plugin>
                 <param name="port">/dev/ttyUSB0</param>
@@ -12,44 +10,44 @@
                 <param name="debug_mode">true</param> <!-- or false -->
             </hardware>
-            <joint name="Joint1">
+            <joint name="joint1">
                 <command_interface name="position"/>
                 <state_interface name="position">
-                  <param name="initial_value">${initial_positions['Joint1']}</param>
+                  <param name="initial_value">${initial_positions['joint1']}</param>
                 </state_interface>
             </joint>
-            <joint name="Joint2">
+            <joint name="joint2">
                 <command_interface name="position"/>
                 <state_interface name="position">
-                  <param name="initial_value">${initial_positions['Joint2']}</param>
+                  <param name="initial_value">${initial_positions['joint2']}</param>
                 </state_interface>
             </joint>
-            <joint name="Joint3">
+            <joint name="joint3">
                 <command_interface name="position"/>
                 <state_interface name="position">
-                  <param name="initial_value">${initial_positions['Joint3']}</param>
+                  <param name="initial_value">${initial_positions['joint3']}</param>
                 </state_interface>
             </joint>
-            <joint name="Joint4">
+            <joint name="joint4">
                 <command_interface name="position"/>
                 <state_interface name="position">
-                  <param name="initial_value">${initial_positions['Joint4']}</param>
+                  <param name="initial_value">${initial_positions['joint4']}</param>
                 </state_interface>
             </joint>
-            <joint name="Joint5">
+            <joint name="joint5">
                 <command_interface name="position"/>
                 <state_interface name="position">
-                  <param name="initial_value">${initial_positions['Joint5']}</param>
+                  <param name="initial_value">${initial_positions['joint5']}</param>
                 </state_interface>
             </joint>
-            <joint name="Joint6">
+            <joint name="joint6">
                 <command_interface name="position"/>
                 <state_interface name="position">
-                  <param name="initial_value">${initial_positions['Joint6']}</param>
+                  <param name="initial_value">${initial_positions['joint6']}</param>
                 </state_interface>
             </joint>
-            <joint name="left_finger">
+            <joint name="right_finger">
                 <command_interface name="position"/>
                 <state_interface name="position">
-                  <param name="initial_value">${initial_positions['left_finger']}</param>
+                  <param name="initial_value">${initial_positions['right_finger']}</param>
                 </state_interface>
             </joint>

File: alicia_duo_moveit/config/alicia_duo_descriptions.urdf.xacro (robot description, xacro)
@@ -6,5 +6,4 @@
     <!-- Import control_xacro -->
     <xacro:include filename="alicia_duo_descriptions.ros2_control.xacro" />
-    <!-- <xacro:alicia_duo_descriptions_ros2_control name="FakeSystem" initial_positions_file="$(arg initial_positions_file)"/> -->
     <xacro:alicia_duo_descriptions_ros2_control name="AliciaDuoSystem" initial_positions_file="$(arg initial_positions_file)"/>
 </robot>
